Commit message: Fix camera color topic bridging

File: bcr_arm_description/urdf/sensors/depth_camera.urdf.xacro (robot description, xacro)
@@ -43,14 +43,16 @@
     <!-- Ignition Gazebo Camera Plugin -->
     <gazebo reference="${prefix}camera_link">
-      <sensor type="camera" name="depth_camera">
-        <always_on>true</always_on>
-        <update_rate>20</update_rate>
-        <visualize>true</visualize>
-        <camera>
-          <horizontal_fov>1.0</horizontal_fov>
-          <image>
-            <width>640</width>
-            <height>480</height>
-            <format>R8G8B8</format>
+        <sensor type="camera" name="depth_camera">
+          <always_on>true</always_on>
+          <update_rate>20</update_rate>
+          <visualize>true</visualize>
+          <topic>/camera/image_raw</topic>
+          <camera_info_topic>/camera/camera_info</camera_info_topic>
+          <camera>
+            <horizontal_fov>1.0</horizontal_fov>
+            <image>
+              <width>640</width>
+              <height>480</height>
+              <format>R8G8B8</format>
           </image>
           <depth_image>
@@ -63,7 +65,7 @@
           </clip>
         </camera>
-        <!-- Sensor data handled by Gazebo sensors system and bridged by ros_gz_bridge -->
-      </sensor>
-    </gazebo>
-  </xacro:macro>
-</robot>
+          <!-- Sensor data handled by Gazebo sensors system and bridged by ros_gz_bridge -->
+        </sensor>
+      </gazebo>
+    </xacro:macro>
+  </robot>
